File: SL&R Overcurrent Analog.brd (EAGLE design)
At the start: 55 x 63.5 mm, 36 parts, among them IC1 TLC393CPN, IC2 CSLA2CFTH, Q3 SUP75P0307, Q4 SUP75P0307, X1 J1, X2 J2, X3 J3

Commit message: Minor updates
Parts:
- renumbered R104 to R4, R105 to R5, R106 to R6, R107 to R7, R108 to R8, R109 to R9
Changed lines of the file:
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@@
 <attribute name="NAME" x="15.666" y="19.579" size="0.9906" layer="25" ratio="10" rot="R90"/>
 </element>
-<element name="R104" library="Overcurrent Detect" package="0204/7" value="3kR" x="3.5" y="26.5" smashed="yes" rot="R270">
+<element name="R4" library="Overcurrent Detect" package="0204/7" value="3kR" x="3.5" y="26.5" smashed="yes" rot="R270">
 <attribute name="NAME" x="4.7954" y="29.04" size="0.9906" layer="25" ratio="10" rot="R270"/>
 </element>
-<element name="R106" library="Overcurrent Detect" package="0204/7" value="2kR" x="5.5" y="17" smashed="yes" rot="R270">
+<element name="R6" library="Overcurrent Detect" package="0204/7" value="2kR" x="5.5" y="17" smashed="yes" rot="R270">
 <attribute name="NAME" x="6.7954" y="19.54" size="0.9906" layer="25" ratio="10" rot="R270"/>
 </element>
-<element name="R108" library="Overcurrent Detect" package="0204/7" value="1MR" x="38" y="26.5" smashed="yes" rot="R90">
+<element name="R8" library="Overcurrent Detect" package="0204/7" value="1MR" x="38" y="26.5" smashed="yes" rot="R90">
 <attribute name="NAME" x="36.7046" y="23.96" size="0.9906" layer="25" ratio="10" rot="R90"/>
 </element>
-<element name="R109" library="Overcurrent Detect" package="0204/7" value="10kR" x="43" y="26.5" smashed="yes" rot="R270">
+<element name="R9" library="Overcurrent Detect" package="0204/7" value="10kR" x="43" y="26.5" smashed="yes" rot="R270">
 <attribute name="NAME" x="44.2954" y="29.04" size="0.9906" layer="25" ratio="10" rot="R270"/>
 </element>
@@
 <attribute name="NAME" x="30.2046" y="35.46" size="0.9906" layer="25" ratio="10" rot="R90"/>
 </element>
-<element name="R105" library="SL&amp;R Overcurrent Analog" package="RTRIM3296W" value="10kR" x="16" y="7.5" smashed="yes">
+<element name="R5" library="SL&amp;R Overcurrent Analog" package="RTRIM3296W" value="10kR" x="16" y="7.5" smashed="yes">
 <attribute name="NAME" x="13.35" y="3" size="0.9906" layer="25" rot="R90"/>
 </element>
@@
 <attribute name="VALUE" x="32.802" y="3.96" size="1.27" layer="27" ratio="10" rot="R90"/>
 </element>
-<element name="R107" library="Overcurrent Detect" package="0204/7" value="10kR" x="12" y="26.5" smashed="yes" rot="R90">
+<element name="R7" library="Overcurrent Detect" package="0204/7" value="10kR" x="12" y="26.5" smashed="yes" rot="R90">
 <attribute name="NAME" x="13.2954" y="29.04" size="0.9906" layer="25" ratio="10" rot="R270"/>
 </element>
@@
 <signal name="+12V">
 <contactref element="R15" pad="2"/>
-<contactref element="R109" pad="2"/>
+<contactref element="R9" pad="2"/>
 <contactref element="X1" pad="1"/>
 <contactref element="IC1" pad="8"/>
@@
 <wire x1="40.5" y1="32" x2="37.15" y2="35.35" width="0.6096" layer="16"/>
 <wire x1="37.15" y1="35.35" x2="37.15" y2="37.5" width="0.6096" layer="16"/>
-<contactref element="R105" pad="3"/>
+<contactref element="R5" pad="3"/>
 <contactref element="R11" pad="2"/>
 <wire x1="5.3882625" y1="23.1517375" x2="7.5" y2="21.04" width="0.6096" layer="16"/>
@@
 <wire x1="46" y1="3.5" x2="29.96" y2="3.5" width="0.6096" layer="16"/>
 <wire x1="29.96" y1="3.5" x2="29.5" y2="3.96" width="0.6096" layer="16"/>
-<contactref element="R107" pad="1"/>
+<contactref element="R7" pad="1"/>
 <contactref element="R13" pad="1"/>
 <wire x1="22.5" y1="4.96" x2="23.96" y2="3.5" width="0.6096" layer="16"/>
@@
 </signal>
 <signal name="N$1">
-<contactref element="R104" pad="2"/>
+<contactref element="R4" pad="2"/>
 <contactref element="IC1" pad="3"/>
-<contactref element="R108" pad="1"/>
+<contactref element="R8" pad="1"/>
 <wire x1="22.27" y1="18.69" x2="22.19" y2="18.69" width="0.6096" layer="16"/>
 <wire x1="5" y1="16" x2="3.5" y2="17.5" width="0.6096" layer="16"/>
@@
 <contactref element="IC1" pad="2"/>
 <contactref element="TP2" pad="P$1"/>
-<contactref element="R106" pad="1"/>
-<contactref element="R107" pad="2"/>
+<contactref element="R6" pad="1"/>
+<contactref element="R7" pad="2"/>
 <wire x1="5.5" y1="20.81" x2="5.5" y2="23.81" width="0.6096" layer="1"/>
 <wire x1="5.5" y1="23.81" x2="12" y2="30.31" width="0.6096" layer="1"/>
@@
 </signal>
 <signal name="N$6">
-<contactref element="R108" pad="2"/>
+<contactref element="R8" pad="2"/>
 <contactref element="IC1" pad="1"/>
 <contactref element="Q3" pad="G"/>
-<contactref element="R109" pad="1"/>
+<contactref element="R9" pad="1"/>
 <contactref element="C2" pad="1"/>
 <contactref element="Q1" pad="2"/>
@@
 <signal name="N$15">
 <contactref element="R10" pad="1"/>
-<contactref element="R104" pad="1"/>
+<contactref element="R4" pad="1"/>
 <contactref element="X2" pad="2"/>
 <contactref element="TP1" pad="P$1"/>
@@
 </signal>
 <signal name="N$20">
-<contactref element="R105" pad="2"/>
-<contactref element="R106" pad="2"/>
+<contactref element="R5" pad="2"/>
+<contactref element="R6" pad="2"/>
 <wire x1="5.5" y1="13.19" x2="5.5" y2="13.25" width="0.6096" layer="16"/>
 <wire x1="5.5" y1="13.25" x2="7.5" y2="11.25" width="0.6096" layer="16"/>
